File: 9key.sch (KiCad schematic (older format))
At the start: 14 parts

Commit message: Add submodules
Parts:
- added C?: 4.7nF, symbol Device:C_Small
- added C? (x3): 0.47uF, symbol Device:C_Small
- added C? (x3): 0.1uF, symbol Device:C_Small
- added C?: 1uF, symbol Device:C_Small
- added D?: D_Schottky_Small, symbol Device:D_Schottky_Small
- added F?: Polyfuse_Small, symbol Device:Polyfuse_Small
- added J?: USB_C_Receptacle_USB2.0, symbol Connector:USB_C_Receptacle_USB2.0
- added MX? (x9): MX-NoLED, symbol MX_Alps_Hybrid:MX-NoLED
- added R? (x2): 5.1k, symbol Device:R_Small_US
- added R?: 1M, symbol Device:R_Small_US
- added R?: 100k, symbol Device:R_Small_US
- added R?: 20k, symbol Device:R_Small_US
- added R?: 1k, symbol Device:R_Small_US
- added R?: 1K, symbol Device:R_Small_US
- added R?: 10k, symbol Device:R_Small_US
- added U?: IS31FL3733-TQ, Package_QFP:TQFP-48-1EP_7x7mm_P0.5mm_EP5x5mm, symbol Driver_LED:IS31FL3733-TQ
- added U?: PRTR5V0U2X, symbol random-keyboard-parts:PRTR5V0U2X
- U?: symbol keeb-rescue:ATmega32U4-AU-MCU_Microchip_ATmega -> MCU_Microchip_ATmega:ATmega32U4-AU
Connections:
- net labels added: SCL, SDA, VBUS
- wire segments 50 -> 169
Other:
- moved on the sheet: C?, R?, SW?, Y?

Commit message: Add submodules
Parts:
- removed MX? (x9): MX-NoLED, symbol MX_Alps_Hybrid:MX-NoLED
- added D10, D2, D3, D4, D5, D6, D7, D8, D9: D_Small, Diode_SMD:D_0201_0603Metric, symbol Device:D_Small
- added J2: Conn_02x05_Odd_Even, symbol Connector_Generic:Conn_02x05_Odd_Even
- added U10, U11, U12, U4, U5, U6, U7, U8, U9: Cherry_MX_RGB, symbol ZOOMER_MX:Cherry_MX_RGB
- C1, C10, C11, C12, C13, C14, C15, C2, C3, C4, C5, C6, C7, C8, C9: renamed from C?; footprint (none) -> Capacitor_SMD:C_0201_0603Metric
- D1: renamed from D?; footprint (none) -> Diode_SMD:D_SOD-123F
- F1: renamed from F?; footprint (none) -> Fuse:Fuse_0805_2012Metric
- gave numbers to parts that had none: 18
Connections:
- net +5V: now also J2.1 (Pin_1)
- net GND: now also J2.4 (Pin_4), J2.7 (Pin_7), J2.9 (Pin_9)
- net MOSI: now reaches U1.10 (PB2)
- net MOSI: now also J2.2 (Pin_2)
- net MISO: now reaches U1.11 (PB3)
- net MISO: now also J2.10 (Pin_10)
- net RST: now reaches R3.2, SW1.2, U1.13 (~RESET)
- net RST: now also J2.6 (Pin_6)
- net C1: now reaches U1.20 (PD2)
- net C1: now also J2.5 (Pin_5), U4.5 (SW1), U5.5 (SW1), U6.5 (SW1)
- net C2: now reaches U1.21 (PD3)
- net C2: now also J2.3 (Pin_3), U7.5 (SW1), U8.5 (SW1), U9.5 (SW1)
- net C3: now reaches U1.25 (PD4)
- net C3: now also U10.5 (SW1), U11.5 (SW1)
- net R3: now reaches U1.39 (PF4)
- net R3: now also D10.1 (K), D4.1 (K), D7.1 (K)
- net R2: now reaches U1.40 (PF1)
- net R2: now also D3.1 (K), D6.1 (K), D9.1 (K)
- net R1: now reaches U1.41 (PF0)
- net R1: now also D2.1 (K), D5.1 (K), D8.1 (K)
- net SCK: now reaches U1.9 (PB1)
- net SCK: now also J2.8 (Pin_8)
- net SW8: now reaches U3.10 (SW8)
- net SW8: now also U12.2 (G-), U6.2 (G-), U9.2 (G-)
- net SW9: now reaches U3.11 (SW9)
- net SW9: now also U12.1 (R-), U6.1 (R-), U9.1 (R-)
- net CS1: now reaches U3.16 (CS1)
- net CS1: now also U4.4 (LED+), U5.4 (LED+), U6.4 (LED+)
- net CS2: now reaches U3.17 (CS2)
- net CS2: now also U7.4 (LED+), U8.4 (LED+), U9.4 (LED+)
- net CS3: now reaches U3.18 (CS3)
- net CS3: now also U10.4 (LED+), U11.4 (LED+), U12.4 (LED+)
- net SW1: now reaches U3.2 (SW1)
- net SW1: now also U10.3 (B-), U4.3 (B-), U7.3 (B-)
- net SW2: now reaches U3.3 (SW2)
- net SW2: now also U10.2 (G-), U4.2 (G-), U7.2 (G-)
- net SW3: now reaches U3.4 (SW3)
- net SW3: now also U10.1 (R-), U4.1 (R-), U7.1 (R-)
- net SW4: now reaches U3.6 (SW4)
- net SW4: now also U11.3 (B-), U5.3 (B-), U8.3 (B-)
- net SW5: now reaches U3.7 (SW5)
- net SW5: now also U11.2 (G-), U5.2 (G-), U8.2 (G-)
- net SW6: now reaches U3.8 (SW6)
- net SW6: now also U11.1 (R-), U5.1 (R-), U8.1 (R-)
- net SW7: now reaches U3.9 (SW7)
- net SW7: now also U12.3 (B-), U6.3 (B-), U9.3 (B-)
- new net: D2.2 (A), U4.6 (SW2)
- new net: D3.2 (A), U5.6 (SW2)
- new net: D4.2 (A), U6.6 (SW2)
- new net: D5.2 (A), U7.6 (SW2)
- new net: D6.2 (A), U8.6 (SW2)
- new net: D7.2 (A), U9.6 (SW2)
- new net: D8.2 (A), U10.6 (SW2)
- new net: D9.2 (A), U11.6 (SW2)
- new net: D10.2 (A), U12.6 (SW2)
Other:
- moved on the sheet: C10, C11, C12, C13, C14, C15, C9, R10, R11, R12, R8, R9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

Commit message: Housekeeping
Updated files included in the project and organized libraries into their own folder.
Parts:
- U10, U11, U12, U4, U5, U6, U7, U8, U9: symbol ZOOMER_MX:Cherry_MX_RGB -> 9key-rescue:Cherry_MX_RGB-ZOOMER_MX
- U2: symbol random-keyboard-parts:PRTR5V0U2X -> 9key-rescue:PRTR5V0U2X-random-keyboard-parts
Connections:
- net C3: now also U12.5 (SW1)
Other:
- note added: "Key Matrix"
- note added: "LED Controller"
- note added: "Microcontroller"
- note added: "USB Interface"
- moved on the sheet: C10, C11, C12, C13, C14, C15, C4, C5, C6, C7, D10, D2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
